File: bubbleclock.sch (KiCad schematic (older format))
At the start: 34 parts, among them J1 Conn_01x01_Male, J2 Conn_01x01_Male, J3 Conn_01x05_Male, J4 14_seg_bubbledisp, Q1 Q_NPN_BEC, Q2 Q_NPN_BEC, SW1 SW_SPDT, U1 ESP-12F, U2 MIC5504-3.3YM5, U3 74HC595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

Commit message: schematic improvements. Board not updated, is broken.
I pulled GPIO15 high instead of low. OOPS!
Connections:
- net +3V3: no longer R5.1
- net AA: now also U3.2 (QC); no longer U3.15 (QA)
- net AB: now also U3.6 (QG); no longer U3.1 (QB)
- net AC: now also U3.15 (QA); no longer U3.2 (QC)
- net AD: now also U3.4 (QE); no longer U3.3 (QD)
- net ADP: now also U3.1 (QB); no longer U3.7 (QH)
- net AE: now also U3.3 (QD); no longer U3.4 (QE)
- net AF: now also U3.7 (QH); no longer U3.5 (QF)
- net AG: now also U3.5 (QF); no longer U3.6 (QG)
- net CS: now also R5.1; no longer R5.2
- net GND: now also R5.2; no longer U1.19 (GPIO4), U1.20 (GPIO5), U1.6 (GPIO12)
- net C1: now reaches J4.1 (C1), U4.15 (QA)
- net C7: now reaches J4.10 (C7), U4.6 (QG)
- net AE': now reaches J4.11 (AE), R12.1
- net C8: now reaches J4.12 (C8), U4.7 (QH)
- net AD': now reaches J4.13 (AD), R11.1
- net C9: now reaches J4.14 (C9), U5.15 (QA)
- net AG': now reaches J4.15 (AG), R14.1
- net C10: now reaches J4.16 (C10), U5.1 (QB)
- net AB': now reaches J4.17 (AB), R9.1
- net C11: now reaches J4.18 (C11), U5.2 (QC)
- net AF': now reaches J4.19 (AF), R13.1
- net C2: now reaches J4.2 (C2), U4.1 (QB)
- net C12: now reaches J4.20 (C12), U5.3 (QD)
- net C13: now reaches J4.21 (C13), U5.4 (QE)
- net C14: now reaches J4.22 (C14), U5.5 (QF)
- net C3: now reaches J4.3 (C3), U4.2 (QC)
- net C4: now reaches J4.4 (C4), U4.3 (QD)
- net AC': now reaches J4.5 (AC), R10.1
- net C5: now reaches J4.6 (C5), U4.4 (QE)
- net ADP': now reaches J4.7 (ADP), R16.1
- net C6: now reaches J4.8 (C6), U4.5 (QF)
- net AA': now reaches J4.9 (AA), R8.1
- net CHAIN1: now reaches U3.9 (QH'), U4.14 (SER)
- net CHAIN2: now reaches U4.9 (QH'), U5.14 (SER)
- net RTS': now reaches Q1.1 (B), R3.1
- net DTR': now reaches Q2.1 (B), R4.1
- no-connect marks 11 -> 14
Other:
- moved on the sheet: R16, R5
Changed lines of the file:
@@
 	7500 2100 7850 2100
 Text Label 7850 1400 2    50   ~ 0
+AC
+Text Label 7850 1500 2    50   ~ 0
+ADP
+Text Label 7850 1600 2    50   ~ 0
 AA
-Text Label 7850 1500 2    50   ~ 0
+Text Label 7850 1700 2    50   ~ 0
+AE
+Text Label 7850 1800 2    50   ~ 0
+AD
+Text Label 7850 1900 2    50   ~ 0
+AG
+Text Label 7850 2000 2    50   ~ 0
 AB
-Text Label 7850 1600 2    50   ~ 0
-AC
-Text Label 7850 1700 2    50   ~ 0
-AD
-Text Label 7850 1800 2    50   ~ 0
-AE
-Text Label 7850 1900 2    50   ~ 0
+Text Label 7850 2100 2    50   ~ 0
 AF
-Text Label 7850 2000 2    50   ~ 0
-AG
-Text Label 7850 2100 2    50   ~ 0
-ADP
 Entry Wire Line
 	7850 1400 7950 1500
@@
 L power:GND #PWR011
 U 1 1 5BFF3AA8
-P 4400 2450
-F 0 "#PWR011" H 4400 2200 50  0001 C CNN
-F 1 "GND" H 4405 2277 50  0000 C CNN
-F 2 "" H 4400 2450 50  0001 C CNN
-F 3 "" H 4400 2450 50  0001 C CNN
-	1    4400 2450
-	1    0    0    -1
-$EndComp
-Wire Wire Line
-	4000 1750 4400 1750
-Wire Wire Line
-	4400 1750 4400 1850
-Wire Wire Line
-	4000 1850 4400 1850
-Connection ~ 4400 1850
-Wire Wire Line
-	4000 1950 4400 1950
-Wire Wire Line
-	4400 1850 4400 1950
-Connection ~ 4400 1950
-Wire Wire Line
-	4400 1950 4400 2450
+P 4450 2750
+F 0 "#PWR011" H 4450 2500 50  0001 C CNN
+F 1 "GND" H 4455 2577 50  0000 C CNN
+F 2 "" H 4450 2750 50  0001 C CNN
+F 3 "" H 4450 2750 50  0001 C CNN
+	1    4450 2750
+	1    0    0    -1
+$EndComp
 Text Label 4250 1450 2    50   ~ 0
 TXD
@@
 CS
 Wire Wire Line
-	4600 2250 4600 2100
-Wire Wire Line
-	4000 2250 4600 2250
+	4000 2250 4450 2250
 $Comp
 L Device:R R5
 U 1 1 5C02C037
-P 4600 1950
-F 0 "R5" H 4670 1996 50  0000 L CNN
-F 1 "10K" H 4670 1905 50  0000 L CNN
-F 2 "Resistor_SMD:R_0805_2012Metric_Pad1.15x1.40mm_HandSolder" V 4530 1950 50  0001 C CNN
-F 3 "~" H 4600 1950 50  0001 C CNN
-	1    4600 1950
-	1    0    0    -1
-$EndComp
-$Comp
-L power:+3V3 #PWR013
-U 1 1 5C02C087
-P 4600 1800
-F 0 "#PWR013" H 4600 1650 50  0001 C CNN
-F 1 "+3V3" H 4615 1973 50  0000 C CNN
-F 2 "" H 4600 1800 50  0001 C CNN
-F 3 "" H 4600 1800 50  0001 C CNN
-	1    4600 1800
+P 4450 2500
+F 0 "R5" H 4520 2546 50  0000 L CNN
+F 1 "10K" H 4520 2455 50  0000 L CNN
+F 2 "Resistor_SMD:R_0805_2012Metric_Pad1.15x1.40mm_HandSolder" V 4380 2500 50  0001 C CNN
+F 3 "~" H 4450 2500 50  0001 C CNN
+	1    4450 2500
 	1    0    0    -1
 $EndComp
@@
 L Device:R R16
 U 1 1 5C280A8A
-P 9450 3000
-F 0 "R16" V 9400 2850 50  0000 C CNN
-F 1 "330" V 9400 3150 50  0000 C CNN
-F 2 "Resistor_SMD:R_0805_2012Metric_Pad1.15x1.40mm_HandSolder" V 9380 3000 50  0001 C CNN
-F 3 "~" H 9450 3000 50  0001 C CNN
-	1    9450 3000
-	0    1    1    0
-$EndComp
-Wire Wire Line
-	9100 3000 9300 3000
-Wire Wire Line
-	9600 3000 9700 3000
+P 9350 3000
+F 0 "R16" V 9350 3000 50  0000 C CNN
+F 1 "330" V 9300 3150 50  0000 C CNN
+F 2 "Resistor_SMD:R_0805_2012Metric_Pad1.15x1.40mm_HandSolder" V 9280 3000 50  0001 C CNN
+F 3 "~" H 9350 3000 50  0001 C CNN
+	1    9350 3000
+	0    1    1    0
+$EndComp
+Wire Wire Line
+	9100 3000 9200 3000
+Wire Wire Line
+	9500 3000 9700 3000
 $Comp
 L power:GND #PWR0101
@@
 Wire Wire Line
 	2650 6200 2950 6200
+Text Label 8850 3200 0    50   ~ 0
+C1
+Text Label 8850 3300 0    50   ~ 0
+C2
+Text Label 8850 3400 0    50   ~ 0
+C3
+Text Label 8850 3500 0    50   ~ 0
+C4
+Text Label 8850 3600 0    50   ~ 0
+C5
+Text Label 8850 3700 0    50   ~ 0
+C6
+Text Label 8850 3800 0    50   ~ 0
+C7
+Text Label 8850 3900 0    50   ~ 0
+C8
+Text Label 8850 4000 0    50   ~ 0
+C9
+Text Label 8850 4100 0    50   ~ 0
+C10
+Text Label 8850 4200 0    50   ~ 0
+C11
+Text Label 8850 4300 0    50   ~ 0
+C12
+Text Label 8850 4400 0    50   ~ 0
+C13
+Text Label 8850 4500 0    50   ~ 0
+C14
+Text Label 9450 2300 0    50   ~ 0
+AA'
+Text Label 9450 2400 0    50   ~ 0
+AB'
+Text Label 9450 2500 0    50   ~ 0
+AC'
+Text Label 9450 2600 0    50   ~ 0
+AD'
+Text Label 9450 2700 0    50   ~ 0
+AE'
+Text Label 9450 2800 0    50   ~ 0
+AF'
+Text Label 9450 2900 0    50   ~ 0
+AG'
+Text Label 9600 3000 0    50   ~ 0
+ADP'
+Text Label 7500 2650 1    50   ~ 0
+CHAIN1
+Text Label 7500 4500 1    50   ~ 0
+CHAIN2
+Text Label 3550 4200 0    50   ~ 0
+RTS'
+Text Label 3550 4800 0    50   ~ 0
+DTR'
+Wire Wire Line
+	4450 2250 4450 2350
+Wire Wire Line
+	4450 2650 4450 2750
+NoConn ~ 4000 1750
+NoConn ~ 4000 1850
+NoConn ~ 4000 1950
 Wire Bus Line
 	7950 1500 7950 2200

Commit message: Redesigned with looser tolerances
Don't torture the boardhouse, plus implementing schematic fixes

Fixes:
1. Pull GPIO0 low instead of high
2. Short regulator enable to VIN
Parts:
- removed J1, J2: Conn_01x01_Male, Connector_PinHeader_2.54mm:PinHeader_1x01_P2.54mm_Vertical, symbol Connector:Conn_01x01_Male
- added J1: Conn_01x02_Male, Connector_PinHeader_2.54mm:PinHeader_1x02_P2.54mm_Vertical, symbol Connector:Conn_01x02_Male
- added R17, R18, R19: 10K, Resistor_SMD:R_0805_2012Metric_Pad1.15x1.40mm_HandSolder, symbol Device:R
- added TP1, TP10, TP2, TP3, TP4, TP5, TP6, TP7, TP8, TP9: TestPoint, TestPoint:TestPoint_Pad_2.5x2.5mm, symbol Connector:TestPoint
- U2: footprint Package_TO_SOT_SMD:SOT-23-5 -> Package_TO_SOT_SMD:SOT-23-5_HandSoldering
Connections:
- net +3V3: now also R17.1, R18.1, R19.1, TP1.1; no longer U1.17 (GPIO2)
- net +BATT: now also J1.1 (Pin_1)
- net GND: now also J1.2 (Pin_2), TP5.1
- net GPIO0: now also TP4.1
- net MOSI: now also TP6.1
- net SCK: now also TP10.1
- net SDA: now reaches U1.19 (GPIO4)
- net SDA: now also R18.2, TP3.1
- net ADC: now reaches U1.2 (ADC)
- net ADC: now also TP9.1
- net SCL: now reaches U1.20 (GPIO5)
- net SCL: now also R19.2, TP7.1
- net MISO: now reaches U1.6 (GPIO12)
- net MISO: now also TP2.1
- net at C2.1, SW1.2 (B), U2.1 (VIN): now also U2.3 (EN)
- new net GPIO2: R17.2, TP8.1, U1.17 (GPIO2)
- no-connect marks 14 -> 9
