File: bubbleclock.kicad_pcb (KiCad board)
At the start: 2 copper layers, 22.9 x 57.2 mm, 46 parts, among them J1 Conn_01x02_Male, J3 Conn_01x05_Male, J4 14_seg_bubbledisp, Q1 Q_NPN_BEC, Q2 Q_NPN_BEC, SW1 SW_SPDT, U1 ESP-12F, U2 MIC5504-3.3YM5, U3 74HC595, U4 74HC595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

Commit message: Minimal tweaks, send to fab!
* Move programming connector down
* Add some sizes
Parts:
- moved J3 1.40 mm to (207.0, 73.2)
- moved R6 1.25 mm to (204.6, 76.5)
- moved R1 1.02 mm to (213.7, 76.3)
- moved R3 1.02 mm to (207.3, 76.3)
- moved R7 1.02 mm to (211.6, 76.3)
- moved R4 1.00 mm to (209.4, 76.3)
Routing:
- net /RESET: track 86.6 -> 84.6 mm
- net /C11: track 22.1 -> 20.6 mm
- net /RTS: track 14.9 -> 13.5 mm
- net Net-(J3-Pad4): track 25.4 -> 24.2 mm
- net /TXD: track 55.3 -> 54.3 mm
- net /DTR': track 2.76 -> 1.76 mm
- net /DTR: track 8.49 -> 7.50 mm
- net /GPIO0: track 34.3 -> 33.3 mm
- net /RTS': track 6.11 -> 5.33 mm
- net /C12: track 21.0 -> 20.4 mm
Other:
- board text added: "DTR"
- board text added: "RTS"
- board text added: "RXD"
- board text added: "TXD"
